File: WeirdBuffer/WeirdBuffer.kicad_sch (KiCad schematic)
At the start: 25 parts

Commit message: second draft
Parts:
- removed D? (x3): LED, symbol Device:LED
- removed J? (x4): Conn_01x02, symbol Connector_Generic:Conn_01x02
- removed R? (x3): LDR03, OptoDevice:R_LDR_10x8.5mm_P7.6mm_Vertical, symbol Sensor_Optical:LDR03
- added C1: 100nF, Capacitor_SMD:C_0805_2012Metric, symbol Device:C
- added D1, D2, D4: LED, LED_THT:LED_D5.0mm, symbol Device:LED
- added J1, J2, J3, J4: AudioJack2_Switch, Connector_Audio:Jack_6.35mm_Neutrik_NMJ4HFD2_Horizontal, symbol Connector:AudioJack2_Switch
- added J5: Conn_02x05_Odd_Even, Connector_IDC:IDC-Header_2x05_P2.54mm_Horizontal, symbol Connector_Generic:Conn_02x05_Odd_Even
- added R10, R12, R9: LDR03, OptoDevice:R_LDR_10x8.5mm_P7.6mm_Vertical, symbol Sensor_Optical:LDR03
- D3: renamed from D?; footprint (none) -> LED_THT:LED_D5.0mm
- R1, R2, R3, R4, R5, R6, R7, R8: renamed from R?; footprint (none) -> Resistor_SMD:R_0805_2012Metric_Pad1.20x1.40mm_HandSolder
- U1: renamed from U?; footprint (none) -> Package_DIP:DIP-14_W7.62mm_LongPads
- gave numbers to parts that had none: 1
Connections:
- net GND: now also D3.1 (K), U1.11 (V-), C1.2, D1.1 (K), D2.1 (K), D4.1 (K), J1.SN, J1.T, J1.TN, J2.SN, J2.T, J2.TN, J3.SN, J3.T, J3.TN, J4.SN, J4.T, J4.TN, J5.2 (Pin_2)
- net at R8.1, U1.2 (-): now also J4.S
- net at R8.2, U1.1: now also D4.2 (A)
- net OUT1B: now reaches R11.2
- net OUT1B: now also J5.4 (Pin_4); no longer D3.1 (K)
- net +5V: now reaches U1.4 (V+)
- net +5V: now also C1.1, J5.1 (Pin_1)
- net at R5.2, U1.8: now also D1.2 (A)
- net at R5.1, U1.9 (-): now also J1.S
- net at R7.1, U1.13 (-): now also J3.S
- net OUT1A: now reaches R11.1
- net OUT1A: now also J5.3 (Pin_3)
- net at R6.2, U1.7: now also D2.2 (A)
- net at R6.1, U1.6 (-): now also J2.S
- new net OUT2A: J5.5 (Pin_5), R12.1
- new net OUT2B: J5.6 (Pin_6), R12.2
- new net OUT3A: J5.7 (Pin_7), R9.1
- new net OUT3B: J5.8 (Pin_8), R9.2
- new net OUT4A: J5.9 (Pin_9), R10.1
- new net OUT4B: J5.10 (Pin_10), R10.2
Other:
- moved on the sheet: D3, R11, U1E

Commit message: add schematic pdf
Other:
- title: (none) -> Optical USB Drum Module
Changed lines of the file:
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@@
 (kicad_sch (version 20211123) (generator eeschema)
   (paper "A4" portrait)
+  (title_block
+    (title "Optical USB Drum Module")
+    (rev "A")
+  )
   (junction (at 62.23 132.08) (diameter 0) (color 0 0 0 0)
   )
